File: AH4.kicad_pcb (KiCad board)
At the start: 2 copper layers, 45 x 71.3 mm, 62 parts, among them J1 USB_C_Receptacle_USB2.0_16P, J2 USB_C_Receptacle_USB2.0_16P, J3 I2CM, J4 AUX1, J5 AP, SW1 SW_DIP_x02, SW2 SW_Push, SW3 AP_I2C_R, SW4 I2CM_R, U1 ICM-45686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

Commit message: update
Parts:
- moved J2 13.7 mm to (217.5, 116.3)
- moved J1 13.0 mm to (204.5, 116.3)
- moved U3 13.0 mm to (204.5, 107.9)
- moved U2 4.46 mm to (199.5, 97.9)
- moved RN1 3.19 mm to (192.2, 95.5)
Routing:
- net /USB_HS-: track 0.00 -> 11.2 mm
- net /USB_HS+: track 0.00 -> 9.67 mm
- net /D1-: track 0.00 -> 7.31 mm
- net /D1+: track 0.10 -> 6.67 mm

Commit message: update
Parts:
- removed D2, D3: Yellow LED, LED_SMD:LED_0603_1608Metric
- added J6: Conn_02x02_Odd_Even, Connector_PinHeader_2.54mm:PinHeader_2x02_P2.54mm_Vertical, F.Cu at (229.2, 106.0)
- added R18: 10k, Resistor_SMD:R_0402_1005Metric, F.Cu at (208.0, 94.8)
- added SW5: BOOTM, Button_Switch_SMD:SW_DIP_SPSTx02_Slide_Copal_CHS-02B_W7.62mm_P1.27mm, F.Cu at (214.3, 99.8)
- C10, C11, C8: value 100nF -> 0.1uF
- D1, D4, D5, D6, D7: footprint LED_SMD:LED_0603_1608Metric -> LED_SMD:LED_0805_2012Metric
- R16: value 1.5k -> 1k
- R6, R7: value 1.5k -> 10k
- Y2: footprint Crystal:Crystal_SMD_2016-4Pin_2.0x1.6mm -> Oscillator:Oscillator_SMD_EuroQuartz_XO32-4Pin_3.2x2.5mm
- moved R4 76.3 mm to (224.0, 113.0)
- moved R10 76.0 mm to (232.1, 74.8)
- moved R9 75.5 mm to (231.5, 91.3)
- moved SW1 73.0 mm to (214.3, 83.0)
- moved R2 66.6 mm to (210.9, 113.5)
- moved R5 64.6 mm to (210.9, 115.3)
- moved R12 63.9 mm to (220.6, 86.2)
- moved R15 63.0 mm to (220.7, 96.3)
- moved R13 62.6 mm to (220.7, 90.8)
- moved R14 62.4 mm to (220.7, 91.8)
- moved D1 59.2 mm to (197.3, 109.0)
- moved R1 56.7 mm to (208.0, 93.8), turned to 180 degrees
- moved Y2 55.7 mm to (204.6, 87.8), turned to 180 degrees
- moved R6 54.3 mm to (208.0, 86.0)
- moved R3 54.0 mm to (198.2, 111.9)
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Connections:
- C12 pad 1: Net-(U2-NRST) -> /NRST
- R1 pad 2: Net-(U2-NRST) -> /NRST
- R17 pad 1: Net-(U2-PB2/BOOT1) -> GND
- R17 pad 2: GND -> /BOOT0
- R6 pad 1: Net-(D3-K) -> /DIP_2
- R7 pad 1: Net-(D2-K) -> /DIP_1
- SW1 pad 1: VDD -> /DIP_1
- SW1 pad 2: VDD -> /DIP_2
- SW1 pad 3: /DIP_2 -> VDD
- SW1 pad 4: /DIP_1 -> VDD
- SW2 pad 2: Net-(U2-NRST) -> /NRST
- U2 pad 25: (no net) -> /FSYNC_EN
- U2 pad 26: /FSYNC_EN -> /INT1
- U2 pad 28: Net-(U2-PB2/BOOT1) -> /BOOT1
- U2 pad 60: unconnected-(U2-BOOT0-Pad60) -> /BOOT0
- U2 pad 7: Net-(U2-NRST) -> /NRST
Routing:
- net /AP_SCK: track 0.00 -> 70.0 mm, vias 0 -> 3
- net /AUX1_MOSI: track 0.00 -> 68.6 mm, vias 0 -> 2
- net /AP_MOSI: track 0.00 -> 66.9 mm, vias 0 -> 3
- net /AUX1_SCK: track 0.00 -> 63.1 mm, vias 0 -> 2
- net /~{AUX1_CS}: track 0.00 -> 46.1 mm, vias 0 -> 2
- net /AUX1_MISO: track 0.00 -> 45.9 mm
- net /AP_MISO: track 0.00 -> 38.4 mm, vias 0 -> 1
- net /~{AP_CS}: track 0.00 -> 32.8 mm
- net /FSYNC: track 0.00 -> 28.1 mm, vias 0 -> 2
- net GND: track 0.00 -> 20.9 mm
- net /TXD: track 0.00 -> 18.9 mm, vias 0 -> 2
- net /RXD: track 0.00 -> 17.6 mm, vias 0 -> 2
- net VDD: track 0.00 -> 14.5 mm
- net /BOOT1: track 0.00 -> 7.63 mm
- net /D2-: track 0.29 -> 7.34 mm, vias 0 -> 2
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Other:
- board size 45 x 71.3 mm -> 45 x 55 mm
- board text added: "AP I2C pullup"
- board text added: "BOOT mode"
- board text added: "BOOT0"
- board text added: "BOOT1"
- board text added: "FSYNC"
- board text added: "GND/3V3"
- board text added: "I2CM pullup"
- board text added: "PWR"
- board text added: "R"
- board text added: "SWC/SWD"
- board text added: "U0"
- board text added: "U1"

Commit message: update
Parts:
- added C16: 0.1uF, Capacitor_SMD:C_0402_1005Metric, F.Cu at (206.8, 93.5)
- added REF**: Linkkalu_v1_5.7x6mm, Logos:Linkkalu_v1_5.7x6mm, F.Cu at (202.0, 69.8)
- J6: value Conn_02x02_Odd_Even -> Prog_conn
- R17: value 10k -> 1k
- SW5: value BOOTM -> Boot; footprint Button_Switch_SMD:SW_DIP_SPSTx02_Slide_Copal_CHS-02B_W7.62mm_P1.27mm -> Button_Switch_SMD:SW_Push_1P1T_NO_Vertical_Wuerth_434133025816
- moved C12 26.1 mm to (218.7, 102.7)
- moved R4 13.6 mm to (211.0, 116.9), turned to 180 degrees
- moved R3 13.1 mm to (211.0, 115.0)
- moved R15 12.5 mm to (208.4, 94.0), turned to 180 degrees
- moved R17 12.5 mm to (201.1, 106.2), turned to 90 degrees
- moved R13 12.4 mm to (208.5, 88.6), turned to 180 degrees
- moved R14 12.4 mm to (208.4, 93.0), turned to 180 degrees
- moved R12 12.2 mm to (208.5, 87.3), turned to 180 degrees
- moved R8 11.6 mm to (201.1, 109.5)
- moved C2 10.8 mm to (206.8, 103.2), turned to 180 degrees
- moved SW2 9.31 mm to (218.7, 99.3)
- moved R16 9.07 mm to (201.1, 108.5)
- moved C14 4.97 mm to (213.8, 73.6)
- moved C15 4.97 mm to (214.9, 73.6)
- moved U1 4.97 mm to (211.3, 75.0)
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Connections:
- R17 pad 2: /BOOT0 -> Net-(U2-BOOT0)
- SW3 pad 1: /AP_MOSI -> Net-(R12-Pad1)
- SW3 pad 2: /AP_SCK -> Net-(R13-Pad1)
- SW3 pad 3: Net-(R13-Pad1) -> /AP_SCK
- SW3 pad 4: Net-(R12-Pad1) -> /AP_MOSI
- SW4 pad 1: /AUX1_MOSI -> Net-(R14-Pad1)
- SW4 pad 2: /AUX1_SCK -> Net-(R15-Pad1)
- SW4 pad 3: Net-(R15-Pad1) -> /AUX1_SCK
- SW4 pad 4: Net-(R14-Pad1) -> /AUX1_MOSI
- SW5 pad 1: /BOOT0 -> /BOOT1
- SW5 pad 2: /BOOT1 -> VDD
- U2 pad 15: unconnected-(U2-PA1/ADC1-Pad15) -> /DIP_1
- U2 pad 16: unconnected-(U2-PA2/ADC2-Pad16) -> /DIP_2
- U2 pad 17: unconnected-(U2-PA3/ADC3-Pad17) -> /FSYNC_EN
- U2 pad 24: /AP_LED -> /FSYNC
- U2 pad 25: /FSYNC_EN -> unconnected-(U2-PC5/ADC15-Pad25)
- U2 pad 27: /FSYNC -> /AP_LED
- U2 pad 60: /BOOT0 -> Net-(U2-BOOT0)
- U2 pad 8: /DIP_1 -> unconnected-(U2-PC0/ADC10-Pad8)
- U2 pad 9: /DIP_2 -> unconnected-(U2-PC1/ADC11-Pad9)
Routing:
- net GND: track 20.9 -> 238.3 mm, vias 0 -> 21
- net VDD: track 14.5 -> 187.1 mm, vias 0 -> 13
- net /OIS_LED: track 0.00 -> 48.1 mm, vias 0 -> 2
- net /I2CM_LED: track 0.00 -> 41.7 mm, vias 0 -> 2
- net Net-(U6-EN): track 0.00 -> 30.7 mm, vias 0 -> 4
- net /AUX1_SCK: track 63.1 -> 91.4 mm
- net /NRST: track 0.00 -> 27.1 mm, vias 0 -> 3
- net /FSYNC_EN: track 0.00 -> 27.1 mm
- net /INT1: track 1.11 -> 24.7 mm, vias 0 -> 2
- net /DIP_1: track 0.00 -> 18.6 mm
- net /BOOT1: track 7.63 -> 25.5 mm, vias 0 -> 3
- net /DIP_2: track 0.00 -> 17.3 mm
- net /AUX1_MOSI: track 68.6 -> 85.6 mm
- net /AP_LED: track 0.00 -> 16.1 mm, vias 0 -> 2
- net Net-(J2-CC2): track 0.00 -> 9.97 mm
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- added copper zone on B.Cu, net GND
- added copper zone on F.Cu, net GND
Other:
- copper layers 2 -> 4
- board text added: "AH4"
- board text added: "B"
- board text added: "CS"
- board text added: "ICM-45658"
- board text added: "UART"
- board text added: "USB"
- board text added: "User mode"
- board text added: "X"
- board text added: "Y"
- board text added: "Z"
- board text removed: "BOOT mode"
- board text removed: "BOOT0"
- board text removed: "BOOT1"
- board text removed: "~{CS}"

Commit message: update
Parts:
- J6: footprint Connector_PinHeader_2.54mm:PinHeader_2x02_P2.54mm_Vertical -> Connector_PinHeader_1.27mm:PinHeader_1x04_P1.27mm_Vertical
- moved J6 3.49 mm to (229.8, 105.6), turned to 0 degrees
Connections:
- J6 pad 2: /SWD -> GND
- J6 pad 3: GND -> /SWD
Routing:
- net /SWD: track 0.00 -> 39.1 mm, vias 0 -> 1
- net /SWC: track 0.00 -> 38.3 mm, vias 0 -> 1
- net VDD: track 187.1 -> 180.6 mm
- net Net-(U6-EN): track 30.7 -> 35.0 mm
- net GND: track 238.3 -> 235.8 mm, vias 21 -> 29
- net Net-(J1-CC1): track 8.60 -> 9.24 mm
- added copper zone on In1.Cu, net GND
- added copper zone on In2.Cu, net GND
- added copper zone on In2.Cu, net VDD
Other:
- board text added: "SWC"
- board text added: "SWD"
- board text removed: "GND/3V3"
- board text removed: "SWC/SWD"

Commit message: update
Routing:
- net GND: track 235.8 -> 252.4 mm, vias 29 -> 62
- net VDD: track 180.6 -> 185.8 mm, vias 13 -> 16
- net /SWC: track 38.3 -> 40.8 mm
- net /SWD: track 39.1 -> 41.4 mm
- net /AUX1_MOSI: track 85.6 -> 86.4 mm
- added copper zone on F.Cu, net VDD
Other:
- board text added: "14.10.2025"

Commit message: update, the board done
Parts:
- added REF**: 4list_1_4x4.4, Logos:4list_1_4x4.4, F.Cu at (221.8, 108.9)
- moved C14 6.26 mm to (207.6, 73.7)
- moved C15 6.26 mm to (208.7, 73.7)
- moved C13 0.57 mm to (211.6, 72.8), turned to 180 degrees
Routing:
- net VDD: track 185.8 -> 126.9 mm
- net GND: track 252.4 -> 216.3 mm, vias 62 -> 67
- net /AUX1_MOSI: track 86.4 -> 67.9 mm
- net /AUX1_SCK: track 91.6 -> 73.6 mm
- net /AUX1_MISO: track 41.5 -> 57.5 mm, vias 0 -> 2
- net /FSYNC: track 37.7 -> 25.5 mm
- net /INT1: track 24.7 -> 34.0 mm
- net /~{AP_CS}: track 30.5 -> 38.8 mm, vias 0 -> 2
- net /OIS_LED: track 48.1 -> 41.5 mm
- net /AP_MOSI: track 60.7 -> 66.1 mm, vias 4 -> 3
- net /AP_SCK: track 70.4 -> 75.2 mm, vias 3 -> 2
- net /~{AUX1_CS}: track 46.8 -> 48.9 mm
- net /AP_MISO: track 38.8 -> 36.8 mm
Other:
- board text added: "Barsotion AH4"
- board text added: "ICM-45686 IMU devboard"

Commit message: update & gerber
Parts:
- renumbered D7 to D2, D4 to D3, D5 to D4, D6 to D5
Routing:
- net VDD: track 126.9 -> 128.8 mm
- net /AUX1_SCK: track 73.6 -> 74.2 mm
- net /AUX1_MOSI: track 67.9 -> 68.4 mm
- net GND: vias 67 -> 68

Commit message: update
Parts:
- C1, C13, C14, C2, C9: value 100nF -> 0.1uF
- R10, R11, R8, R9: value 1.5k -> 1k
Changed lines of the file:
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@@
 		(allow_soldermask_bridges_in_footprints no)
 		(tenting front back)
+		(aux_axis_origin 189 120)
 		(grid_origin 189 120)
 		(pcbplotparams
@@
 			)
 		)
-		(property "Value" "1.5k"
+		(property "Value" "1k"
 			(at 0 1.17 0)
 			(layer "F.Fab")
@@
 			)
 		)
-		(property "Description" "Light emitting diode"
+		(property "Description" "Light emitting diode, red 0805"
 			(at 0 0 90)
 			(layer "F.Fab")
@@
 			)
 		)
-		(property "Description" "Light emitting diode"
+		(property "Description" "Light emitting diode, red 0805"
 			(at 0 0 90)
 			(layer "F.Fab")
@@
 		(sheetname "/")
 		(sheetfile "AH4.kicad_sch")
-		(attr through_hole)
+		(attr through_hole exclude_from_bom)
 		(fp_line
 			(start -1.38 -1.38)
@@
 			)
 		)
-		(property "Value" "1.5k"
+		(property "Value" "1k"
 			(at 0 1.17 0)
 			(layer "F.Fab")
@@
 			)
 		)
-		(property "Description" ""
+		(property "Description" "RISC-V WCH MCU"
 			(at 0 0 0)
 			(layer "F.Fab")
@@
 			)
 		)
-		(property "Value" "100nF"
+		(property "Value" "0.1uF"
 			(at 0 1.16 0)
 			(layer "F.Fab")
@@
 			)
 		)
-		(property "Description" "Light emitting diode"
+		(property "Description" "Light emitting diode, yellow 0805"
 			(at 0 0 0)
 			(layer "F.Fab")
@@
 			)
 		)
-		(property "Description" "Light emitting diode"
+		(property "Description" "Light emitting diode, red 0805"
 			(at 0 0 90)
 			(layer "F.Fab")
@@
 			)
 		)
-		(property "Value" "100nF"
+		(property "Value" "0.1uF"
 			(at 0 1.16 0)
 			(layer "F.Fab")
@@
 			)
 		)
-		(property "Value" "100nF"
+		(property "Value" "0.1uF"
 			(at 0 1.16 0)
 			(layer "F.Fab")
@@
 		(sheetname "/")
 		(sheetfile "AH4.kicad_sch")
-		(attr through_hole)
+		(attr through_hole exclude_from_bom)
 		(fp_line
 			(start 1.38 1.27)
@@
 			)
 		)
-		(property "Value" "100nF"
+		(property "Value" "0.1uF"
 			(at 0 1.16 90)
 			(layer "F.Fab")
@@
 			)
 		)
-		(property "Value" "1.5k"
+		(property "Value" "1k"
 			(at 0 1.17 0)
 			(layer "F.Fab")
@@
 			)
 		)
-		(property "Description" ""
+		(property "Description" "Inertial measurement unit"
 			(at -15.45 5.25 0)
 			(unlocked yes)
@@
 		(sheetname "/")
 		(sheetfile "AH4.kicad_sch")
-		(attr through_hole)
+		(attr through_hole exclude_from_bom)
 		(fp_line
 			(start 1.38 1.27)
@@
 			)
 		)
-		(property "Description" "Light emitting diode"
+		(property "Description" "Light emitting diode, yellow 0805"
 			(at 0 0 0)
 			(layer "F.Fab")
@@
 			)
 		)
-		(property "Value" "1.5k"
+		(property "Value" "1k"
 			(at 0 1.17 0)
 			(layer "F.Fab")
@@
 			)
 		)
-		(property "Value" "100nF"
+		(property "Value" "0.1uF"
 			(at 0 1.16 90)
 			(layer "F.Fab")
