File: AH4.kicad_sch (KiCad schematic)
At the start: 62 parts, among them J1 USB_C_Receptacle_USB2.0_16P, J2 USB_C_Receptacle_USB2.0_16P, J3 I2CM, J4 AUX1, J5 AP, SW1 SW_DIP_x02, SW2 SW_Push, SW3 AP_I2C_R, SW4 I2CM_R, U1 ICM-45686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

Commit message: update
Parts:
- removed D2, D3: Yellow LED, LED_SMD:LED_0603_1608Metric, symbol Device:LED
- added J6: Conn_02x02_Odd_Even, Connector_PinHeader_2.54mm:PinHeader_2x02_P2.54mm_Vertical, symbol Connector_Generic:Conn_02x02_Odd_Even
- added R18: 10k, Resistor_SMD:R_0402_1005Metric, symbol Device:R
- added SW5: BOOTM, Button_Switch_SMD:SW_DIP_SPSTx02_Slide_Copal_CHS-02B_W7.62mm_P1.27mm, symbol Switch:SW_DIP_x02
- C10, C11, C8: value 100nF -> 0.1uF
- D1, D4, D5, D6, D7: footprint LED_SMD:LED_0603_1608Metric -> LED_SMD:LED_0805_2012Metric
- R16: value 1.5k -> 1k
- R6, R7: value 1.5k -> 10k
- Y2: footprint Crystal:Crystal_SMD_2016-4Pin_2.0x1.6mm -> Oscillator:Oscillator_SMD_EuroQuartz_XO32-4Pin_3.2x2.5mm
Connections:
- net DIP_1: now also R7.1, SW1.1; no longer SW1.4
- net DIP_2: now also R6.1, SW1.2; no longer SW1.3
- net FSYNC_EN: now also U2.25 (PC5/ADC15); no longer U2.26 (PB0/ADC8)
- net GND: now also R17.1, J6.3 (Pin_3), R18.2; no longer R17.2
- net NRST: now also C12.1, R1.2, SW2.2, U2.7 (NRST)
- net SWC: now also J6.4 (Pin_4)
- net SWD: now also J6.2 (Pin_2)
- net VDD: now also SW1.3, SW1.4, J6.1 (Pin_1), SW5.3, SW5.4; no longer SW1.1, SW1.2
- net BOOT1: now reaches U2.28 (PB2/BOOT1)
- net BOOT1: now also R18.1, SW5.2; no longer R17.1
- net BOOT0: now reaches U2.60 (BOOT0)
- net BOOT0: now also R17.2, SW5.1
- no-connect marks 37 -> 36
Other:
- moved on the sheet: C12, C13, C14, C15, C5, C6, J3, J4, J5, R1, R17, R6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

Commit message: update
Parts:
- removed SW5: BOOTM, Button_Switch_SMD:SW_DIP_SPSTx02_Slide_Copal_CHS-02B_W7.62mm_P1.27mm, symbol Switch:SW_DIP_x02
- added C16: 0.1uF, Capacitor_SMD:C_0402_1005Metric, symbol Device:C
- added SW5: Boot, Button_Switch_SMD:SW_Push_1P1T_NO_Vertical_Wuerth_434133025816, symbol Switch:SW_Push
- J6: value Conn_02x02_Odd_Even -> Prog_conn
- R17: value 10k -> 1k
Connections:
- net AP_LED: now also U2.27 (PB1/ADC9); no longer U2.24 (PC4/ADC14)
- net AP_MOSI: now also SW3.4; no longer SW3.1
- net AP_SCK: now also SW3.3; no longer SW3.2
- net AUX1_MOSI: now also SW4.4; no longer SW4.1
- net AUX1_SCK: now also SW4.3; no longer SW4.2
- net BOOT1: now also C16.2, SW5.1
- net DIP_1: now also U2.15 (PA1/ADC1); no longer U2.8 (PC0/ADC10)
- net DIP_2: now also U2.16 (PA2/ADC2); no longer U2.9 (PC1/ADC11)
- net FSYNC: now also U2.24 (PC4/ADC14); no longer U2.27 (PB1/ADC9)
- net FSYNC_EN: now also U2.17 (PA3/ADC3); no longer U2.25 (PC5/ADC15)
- net VDD: now also C16.1, SW5.2
- net at R15.1: now also SW4.2; no longer SW4.3
- net at R14.1: now also SW4.1; no longer SW4.4
- net at R12.1: now also SW3.1; no longer SW3.4
- net at R13.1: now also SW3.2; no longer SW3.3
- net BOOT0: no longer names the net of R17.2, U2.60 (BOOT0)

Commit message: update
Parts:
- removed J6: Prog_conn, Connector_PinHeader_2.54mm:PinHeader_2x02_P2.54mm_Vertical, symbol Connector_Generic:Conn_02x02_Odd_Even
- added J6: Prog_conn, Connector_PinHeader_1.27mm:PinHeader_1x04_P1.27mm_Vertical, symbol Connector:Conn_01x04_Pin
Connections:
- net GND: now also J6.2 (Pin_2)
- net SWC: now also J6.4 (Pin_4)
- net SWD: now also J6.3 (Pin_3)
- net VDD: now also J6.1 (Pin_1)
Other:
- moved on the sheet: C16, SW5

Commit message: update & gerber
Parts:
- C1, C13, C14, C2, C9: value 100nF -> 0.1uF
- J1, J2: Mfr.Part (none) -> TYPE C-DB-116PWB
- J3, J4, J5: now left out of the parts list
- SW1, SW3, SW4: Mfr.Part CHS-02TB1 -> CHS-02TB1
- U1: Mfr.Part (none) -> ICM-45686
- U3, U4: Mfr.Part (none) -> USBLC6-2SC6
- U5: Mfr.Part (none) -> CH340X
- U6: Mfr.Part (none) -> AP2112K-3.3TRG1
- renumbered D7 to D2, D4 to D3, D5 to D4, D6 to D5
Changed lines of the file:
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@@
 		(title "Barsotion AH4 - ICM-45686 devboard")
 		(date "2025-10-14")
-		(rev "1.4")
+		(rev "1.5")
 		(company "Barsotion KOy")
 		(comment 1 "Barsy-Barsevich")
@@
 			)
 		)
-		(property "Description" "Light emitting diode"
+		(property "Description" "Light emitting diode, yellow 0805"
 			(at 124.46 177.8 0)
 			(effects
@@
 		(unit 1)
 		(exclude_from_sim no)
-		(in_bom yes)
+		(in_bom no)
 		(on_board yes)
 		(dnp no)
@@
 			)
 		)
-		(property "Value" "100nF"
+		(property "Value" "0.1uF"
 			(at 208.534 50.292 0)
 			(effects
@@
 			)
 		)
+		(property "Mfr.Part" "CH340X"
+			(at 41.91 139.7 0)
+			(effects
+				(font
+					(size 1.27 1.27)
+				)
+				(hide yes)
+			)
+		)
 		(pin "3"
 		)
@@
 			)
 		)
-		(property "Mfr.Part" "   CHS-02TB1 "
+		(property "Mfr.Part" "CHS-02TB1 "
 			(at 255.27 41.91 0)
 			(effects
@@
 			)
 		)
-		(property "Description" ""
+		(property "Description" "RISC-V WCH MCU"
 			(at 172.72 63.5 0)
 			(effects
@@
 		(on_board yes)
 		(dnp no)
-		(property "Reference" "D6"
+		(property "Reference" "D5"
 			(at 39.37 177.038 0)
 			(effects
@@
 			)
 		)
-		(property "Description" "Light emitting diode"
+		(property "Description" "Light emitting diode, red 0805"
 			(at 39.37 180.34 0)
 			(effects
@@
 			(project "AH4"
 				(path "/9bb009d6-2388-4e89-bd21-3189acc261ba"
-					(reference "D6")
+					(reference "D5")
 					(unit 1)
 				)
@@
 			)
 		)
+		(property "Mfr.Part" "USBLC6-2SC6"
+			(at 69.85 90.17 0)
+			(effects
+				(font
+					(size 1.27 1.27)
+				)
+				(hide yes)
+			)
+		)
 		(pin "6"
 		)
@@
 		(unit 1)
 		(exclude_from_sim no)
-		(in_bom yes)
+		(in_bom no)
 		(on_board yes)
 		(dnp no)
@@
 		(on_board yes)
 		(dnp no)
-		(property "Reference" "D5"
+		(property "Reference" "D4"
 			(at 39.37 170.688 0)
 			(effects
@@
 			)
 		)
-		(property "Description" "Light emitting diode"
+		(property "Description" "Light emitting diode, red 0805"
 			(at 39.37 173.99 0)
 			(effects
@@
 			(project "AH4"
 				(path "/9bb009d6-2388-4e89-bd21-3189acc261ba"
-					(reference "D5")
+					(reference "D4")
 					(unit 1)
 				)
@@
 			)
 		)
-		(property "Mfr.Part" "   CHS-02TB1 "
+		(property "Mfr.Part" "CHS-02TB1 "
 			(at 255.27 26.67 0)
 			(effects
@@
 			)
 		)
-		(property "Value" "100nF"
+		(property "Value" "0.1uF"
 			(at 134.62 152.4 0)
 			(effects
@@
 			)
 		)
-		(property "Value" "100nF"
+		(property "Value" "0.1uF"
 			(at 67.056 152.654 90)
 			(effects
@@
 			)
 		)
+		(property "Mfr.Part" "TYPE C-DB-116PWB"
+			(at 34.29 43.18 0)
+			(effects
+				(font
+					(size 1.27 1.27)
+				)
+				(hide yes)
+			)
+		)
 		(pin "S1"
 		)
@@
 			)
 		)
-		(property "Mfr.Part" "   CHS-02TB1 "
+		(property "Mfr.Part" "CHS-02TB1 "
 			(at 92.71 176.53 0)
 			(effects
@@
 			)
 		)
+		(property "Mfr.Part" "AP2112K-3.3TRG1"
+			(at 100.33 30.48 0)
+			(effects
+				(font
+					(size 1.27 1.27)
+				)
+				(hide yes)
+			)
+		)
 		(pin "2"
 		)
@@
 			)
 		)
+		(property "Mfr.Part" "USBLC6-2SC6"
+			(at 69.85 40.64 0)
+			(effects
+				(font
+					(size 1.27 1.27)
+				)
+				(hide yes)
+			)
+		)
 		(pin "6"
 		)
@@
 			)
 		)
-		(property "Value" "100nF"
+		(property "Value" "0.1uF"
 			(at 201.422 50.292 0)
 			(effects
@@
 		(unit 1)
 		(exclude_from_sim no)
-		(in_bom yes)
+		(in_bom no)
 		(on_board yes)
 		(dnp no)
@@
 		(on_board yes)
 		(dnp no)
-		(property "Reference" "D7"
+		(property "Reference" "D2"
 			(at 101.092 88.9 90)
 			(effects
@@
 			)
 		)
-		(property "Description" "Light emitting diode"
+		(property "Description" "Light emitting diode, yellow 0805"
 			(at 97.79 88.9 0)
 			(effects
@@
 			(project "AH4"
 				(path "/9bb009d6-2388-4e89-bd21-3189acc261ba"
-					(reference "D7")
+					(reference "D2")
 					(unit 1)
 				)
@@
 		(on_board yes)
 		(dnp no)
-		(property "Reference" "D4"
+		(property "Reference" "D3"
 			(at 39.37 164.338 0)
 			(effects
@@
 			)
 		)
-		(property "Description" "Light emitting diode"
+		(property "Description" "Light emitting diode, red 0805"
 			(at 39.37 167.64 0)
 			(effects
@@
 			(project "AH4"
 				(path "/9bb009d6-2388-4e89-bd21-3189acc261ba"
-					(reference "D4")
+					(reference "D3")
 					(unit 1)
 				)
@@
 			)
 		)
-		(property "Description" ""
+		(property "Description" "Inertial measurement unit"
+			(at 162.56 38.1 0)
+			(effects
+				(font
+					(size 1.27 1.27)
+				)
+				(hide yes)
+			)
+		)
+		(property "Mfr.Part" "ICM-45686"
 			(at 162.56 38.1 0)
 			(effects
@@
 			)
 		)
+		(property "Mfr.Part" "TYPE C-DB-116PWB"
+			(at 34.29 92.71 0)
+			(effects
+				(font
+					(size 1.27 1.27)
+				)
+				(hide yes)
+			)
+		)
 		(pin "S1"
 		)
@@
 			)
 		)
-		(property "Value" "100nF"
+		(property "Value" "0.1uF"
 			(at 60.96 140.9699 0)
 			(effects

Commit message: update
Parts:
- R10, R11, R8, R9: value 1.5k -> 1k
Changed lines of the file:
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@@
 	(title_block
 		(title "Barsotion AH4 - ICM-45686 devboard")
-		(date "2025-10-14")
-		(rev "1.5")
+		(date "2025-10-15")
+		(rev "1.6")
 		(company "Barsotion KOy")
 		(comment 1 "Barsy-Barsevich")
+		(comment 2 "rev1.6: 1.5k resistors became 1k")
 	)
 	(junction
@@
 			)
 		)
-		(property "Value" "1.5k"
+		(property "Value" "1k"
 			(at 126.238 185.42 0)
 			(effects
@@
 			)
 		)
-		(property "Value" "1.5k"
+		(property "Value" "1k"
 			(at 52.832 177.546 90)
 			(effects
@@
 			)
 		)
-		(property "Value" "1.5k"
+		(property "Value" "1k"
 			(at 52.832 164.846 90)
 			(effects
@@
 			)
 		)
-		(property "Value" "1.5k"
+		(property "Value" "1k"
 			(at 52.832 171.196 90)
 			(effects
